File: axp192breakout.kicad_pcb (KiCad board)
At the start: 2 copper layers, 30.5 x 30.5 mm, 28 parts, among them J1 USB_B_Micro, J2 Conn_02x06_Odd_Even, J3 Conn_01x02, J4 Conn_01x03, J5 Conn_02x08_Odd_Even, J6 Conn_01x03, SW1 SW_SPST, U1 axp192

Commit message: Fix soldermask. Add rendered gerbers. Add rendered schematic.
Other:
- rule pad_to_mask_clearance: 0.051 -> 0
Changed lines of the file:
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@@
     (pad_size 1.524 1.524)
     (pad_drill 0.762)
-    (pad_to_mask_clearance 0.051)
-    (solder_mask_min_width 0.25)
+    (pad_to_mask_clearance 0)
     (aux_axis_origin 0 0)
     (visible_elements FFFFFF7F)
@@
       (outputformat 1)
       (mirror false)
-      (drillshape 1)
+      (drillshape 0)
       (scaleselection 1)
-      (outputdirectory ""))
+      (outputdirectory "gerbers/"))
   )
   (net 0 "")
@@
     (add_net "Net-(D1-Pad2)")
     (add_net "Net-(J1-Pad2)")
-    (add_net "Net-(J1-Pad4)")
     (add_net "Net-(J1-Pad6)")
     (add_net "Net-(J6-Pad2)")
